Commit message: Change joint type

File: src/robot_description/urdf/robot.urdf.xacro (robot description, xacro)
@@ -31,5 +31,5 @@
         <xacro:property name="link_5_radius" value="0.05" />
         <xacro:property name="link_5_length" value="0.03" />
-        <xacro:property name="end_effector_length" value="0.01" />
+        <xacro:property name="end_effector_length" value="0.005" />
         <xacro:property name="end_effector_width" value="0.005" />
         <xacro:property name="end_effector_height" value="0.005" />
@@ -146,5 +146,6 @@
             mass="0.5"
             colour="bone" />
-        <joint name="joint_4" type="continuous">
+        <joint name="joint_4" type="revolute">
+            <limit lower="${-pi}" upper="${pi}" effort="0.0" velocity="${pi}" />
             <parent link="link_3" />
             <child link="link_4" />
